File: tlcs_1-6.sch (KiCad schematic (older format))
At the start: 66 parts, among them U3 TLC5941, U4 TLC5941, U5 TLC5941, U6 TLC5941, U7 TLC5941, U8 TLC5941

Commit message: opened in KiCAD 5.1.4 and went through rescue process
seems to have moved all parts to tca-rescue lib, updated EESchema Library version and removed references to default libs. OK for now so can work on, may adjust libraries later. not committed 'rescue-backup' folder, don't need this when under version control.
Parts:
- C10, C11, C6, C7, C8, C9: symbol C -> tca-rescue:C
- D1, D10, D11, D12, D13, D14, D15, D16, D17, D18, D19, D2, D20, D21, D22, D23, D24, D25, D26, D27, D28, D29, D3, D30, D31, D32, D33, D34, D35, D36, D37, D38, D39, D4, D40, D41, D42, D43, D44, D45, D46, D47, D48, D5, D6, D7, D8, D9: symbol DOUBLE_LED_SEP -> tca-rescue:DOUBLE_LED_SEP
- R3, R4, R5, R6, R7, R8: symbol R -> tca-rescue:R
- U3, U4, U5, U6, U7, U8: symbol TLC5941 -> tca-rescue:TLC5941
