File: tlcs_1-6.sch (KiCad schematic (older format))
At the start: 115 parts, among them U3 TLC5941, U4 TLC5941, U5 TLC5941, U6 TLC5941, U7 TLC5941, U8 TLC5941

Commit message: library work, connect regulator VCC, change value of decoupling caps to be in terms of nF
changed all 0.1uF caps to be 100nF (same, but more common expression)
set pin4 of regulator to be VCC and connected up (can't be sure without source BOM, but think pin2 is NC and footprint/symbol has been done poorly
move all remaining grounds and capacitors to use main KiCAD library symbols, and deleted all remnants of rescue library
exported all remaining footprints from PCB and put in footprint library, and changed footprint references to point there so now all valid
also copied input capacitor footprint to library so I can customise with correct 3D model
changed input inductor footprint (realised previous "1210" was actually 1206!) - copied a generic SMD-1210 footprint from KiCAD libraries to my library and named L-1210 and attached 3d model
changed LED driver TLC5941 footprint in library so pin29 (thermal pad) is solid connection
added 3d model for the resonator, just guessed at one of similar size, used AWSCR-CV step model from abracon website
Parts:
- C10, C11, C6, C7, C8, C9: value 0.1 uF -> 100nF; symbol tca-rescue:C -> Device:C
- C12: symbol tca-rescue:C -> Device:C
Changed lines of the file:
@@
 $EndComp
 $Comp
-L tca-rescue:C C8
+L Device:C C8
 U 1 1 53630180
 P 4050 5400
 F 0 "C8" H 4050 5500 40  0000 L CNN
-F 1 "0.1 uF" H 4056 5315 40  0000 L CNN
+F 1 "100nF" H 4056 5315 40  0000 L CNN
 F 2 "Capacitors_SMD:C_0805" H 4088 5250 30  0001 C CNN
 F 3 "~" H 4050 5400 60  0000 C CNN
@@
 $EndComp
 $Comp
-L tca-rescue:C C7
+L Device:C C7
 U 1 1 53AA0807
 P 4050 3050
 F 0 "C7" H 4050 3150 40  0000 L CNN
-F 1 "0.1 uF" H 4056 2965 40  0000 L CNN
+F 1 "100nF" H 4056 2965 40  0000 L CNN
 F 2 "Capacitors_SMD:C_0805" H 4088 2900 30  0001 C CNN
 F 3 "~" H 4050 3050 60  0000 C CNN
@@
 NoConn ~ 3750 1500
 $Comp
-L tca-rescue:GND #PWR012
+L power:GND #PWR012
 U 1 1 53630970
 P 2050 1000
@@
 $EndComp
 $Comp
-L tca-rescue:C C6
+L Device:C C6
 U 1 1 53630972
 P 4050 800
 F 0 "C6" H 4050 900 40  0000 L CNN
-F 1 "0.1 uF" H 4056 715 40  0000 L CNN
+F 1 "100nF" H 4056 715 40  0000 L CNN
 F 2 "Capacitors_SMD:C_0805" H 4088 650 30  0001 C CNN
 F 3 "~" H 4050 800 60  0000 C CNN
@@
 $EndComp
 $Comp
-L tca-rescue:C C11
+L Device:C C11
 U 1 1 53630EAA
 P 9600 4750
 F 0 "C11" H 9600 4850 40  0000 L CNN
-F 1 "0.1 uF" H 9606 4665 40  0000 L CNN
+F 1 "100nF" H 9606 4665 40  0000 L CNN
 F 2 "Capacitors_SMD:C_0805" H 9638 4600 30  0001 C CNN
 F 3 "~" H 9600 4750 60  0000 C CNN
@@
 $EndComp
 $Comp
-L tca-rescue:C C9
+L Device:C C9
 U 1 1 53630EE2
 P 9600 750
 F 0 "C9" H 9600 850 40  0000 L CNN
-F 1 "0.1 uF" H 9606 665 40  0000 L CNN
+F 1 "100nF" H 9606 665 40  0000 L CNN
 F 2 "Capacitors_SMD:C_0805" H 9638 600 30  0001 C CNN
 F 3 "~" H 9600 750 60  0000 C CNN
@@
 	1300 3750 1300 3850
 $Comp
-L tca-rescue:GND #PWR010
+L power:GND #PWR010
 U 1 1 5DBCA392
 P 2050 3250
@@
 Wire Wire Line
 	1300 6100 1300 6200
-$Comp
-L tca-rescue:GND #PWR08
-U 1 1 5DE22866
-P 2050 5600
-F 0 "#PWR08" H 2050 5600 30  0001 C CNN
-F 1 "GND" H 2050 5530 30  0001 C CNN
-F 2 "" H 2050 5600 60  0000 C CNN
-F 3 "" H 2050 5600 60  0000 C CNN
-	1    2050 5600
-	0    1    1    0
-$EndComp
 Text HLabel 1250 6100 0    60   Input ~ 0
 VIN
@@
 GSCLK
 $Comp
-L tca-rescue:C C10
+L Device:C C10
 U 1 1 53630EC9
 P 9600 2750
 F 0 "C10" H 9600 2850 40  0000 L CNN
-F 1 "0.1 uF" H 9606 2665 40  0000 L CNN
+F 1 "100nF" H 9606 2665 40  0000 L CNN
 F 2 "Capacitors_SMD:C_0805" H 9638 2600 30  0001 C CNN
 F 3 "~" H 9600 2750 60  0000 C CNN
@@
 	6850 1450 6850 1550
 $Comp
-L tca-rescue:GND #PWR014
+L power:GND #PWR014
 U 1 1 5D9616E2
 P 7600 950
@@
 	6850 3450 6850 3550
 $Comp
-L tca-rescue:GND #PWR016
+L power:GND #PWR016
 U 1 1 5D9F850C
 P 7600 2950
@@
 	6850 5450 6850 5550
 $Comp
-L tca-rescue:GND #PWR018
+L power:GND #PWR018
 U 1 1 5DAA6638
 P 7600 4950
@@
 	1650 2650 5200 2650
 $Comp
-L tca-rescue:C C?
+L Device:C C?
 U 1 1 5D98BF30
 P 5750 6850
@@
 	1    0    0    -1
 $EndComp
-Wire Wire Line
-	5750 7050 5750 7100
 Text HLabel 5700 6550 0    60   Input ~ 0
 VCC
 Wire Wire Line
 	5700 6550 5750 6550
-Wire Wire Line
-	5750 6550 5750 6650
 $Comp
 L power:GND #PWR0114
@@
 Wire Wire Line
 	9300 1050 9600 1050
+Wire Wire Line
+	5750 7000 5750 7100
+Wire Wire Line
+	5750 6550 5750 6700
+Wire Wire Line
+	4050 5200 4050 5250
+Wire Wire Line
+	4050 5550 4050 5600
+Wire Wire Line
+	4050 2850 4050 2900
+Wire Wire Line
+	4050 3200 4050 3250
+Wire Wire Line
+	4050 600  4050 650
+Wire Wire Line
+	4050 950  4050 1000
+Wire Wire Line
+	9600 550  9600 600
+Wire Wire Line
+	9600 900  9600 950
+Wire Wire Line
+	9600 2550 9600 2600
+Wire Wire Line
+	9600 2900 9600 2950
+Wire Wire Line
+	9600 4550 9600 4600
+Wire Wire Line
+	9600 4900 9600 4950
+$Comp
+L power:GND #PWR08
+U 1 1 5DE22866
+P 2050 5600
+F 0 "#PWR08" H 2050 5600 30  0001 C CNN
+F 1 "GND" H 2050 5530 30  0001 C CNN
+F 2 "" H 2050 5600 60  0000 C CNN
+F 3 "" H 2050 5600 60  0000 C CNN
+	1    2050 5600
+	0    1    1    0
+$EndComp
 $EndSCHEMATC
