File: tlcs_7-12.sch (KiCad schematic (older format))
At the start: 66 parts, among them U10 TLC5941, U11 TLC5941, U12 TLC5941, U13 TLC5941, U14 TLC5941, U9 TLC5941

Commit message: opened in KiCAD 5.1.4 and went through rescue process
seems to have moved all parts to tca-rescue lib, updated EESchema Library version and removed references to default libs. OK for now so can work on, may adjust libraries later. not committed 'rescue-backup' folder, don't need this when under version control.
Parts:
- C12, C13, C14, C15, C16, C17: symbol C -> tca-rescue:C
- D49, D50, D51, D52, D53, D54, D55, D56, D57, D58, D59, D60, D61, D62, D63, D64, D65, D66, D67, D68, D69, D70, D71, D72, D73, D74, D75, D76, D77, D78, D79, D80, D81, D82, D83, D84, D85, D86, D87, D88, D89, D90, D91, D92, D93, D94, D95, D96: symbol DOUBLE_LED_SEP -> tca-rescue:DOUBLE_LED_SEP
- R10, R11, R12, R13, R14, R9: symbol R -> tca-rescue:R
- U10, U11, U12, U13, U14, U9: symbol TLC5941 -> tca-rescue:TLC5941
